File: hardware/pcb/carrier/carrier.kicad_pcb (KiCad board)
At the start: 2 copper layers, 66 x 54 mm, 38 parts

Commit message: still working on it
Parts:
- removed the C_SDIN at (25.0, 16.0)
- removed the C_SDOUT at (25.0, 24.0)
- removed the C_SDSOCKET at (10.0, 43.0)
- added C_SDIN: 4.7uF X7R 16V, Carrier:C_0805_Murata, F.Cu at (25.0, 16.0)
- added C_SDOUT: 4.7uF X7R 16V, Carrier:C_0805_Murata, F.Cu at (25.0, 24.0)
- added C_SDSOCKET: 100nF X7R 16V, Carrier:C_0805_Murata, F.Cu at (10.0, 43.0)
- C1, C2: footprint Carrier:C_0805 -> Carrier:C_0805_Murata
- C_SDBULK: value 22uF X7R 16V -> 22uF X5R 16V
