File: hardware/pcb/carrier/carrier.kicad_sch (KiCad schematic)
At the start: 34 parts

Commit message: still working on it
Parts:
- C1, C_SDSOCKET: footprint Carrier:C_0805 -> Carrier:C_0805_Murata; MPN (none) -> GRM21BR71C104KA01L
- C2: footprint Carrier:C_0805 -> Carrier:C_0805_Murata; MPN (none) -> GRM21BR71C105KA01L
- C_SDBULK: value 22uF X7R 16V -> 22uF X5R 16V; MPN (none) -> CL31A226KOHNNNE
- C_SDIN, C_SDOUT: footprint Carrier:C_0805 -> Carrier:C_0805_Murata; MPN (none) -> GRM21BR71C475KA73L
- D1, D2, D3, D4, D5: MPN (none) -> APT2012LZGCK
- J_EVM: MPN (none) -> NPPN062FJFN-RC
- J_PICO: MPN (none) -> Pico 2 W
- J_SD: MPN (none) -> 693072010801
- J_UART: MPN (none) -> B5B-XH-A(LF)(SN)
- R_CS, R_PD1, R_PD2, R_PD3, R_PD4, R_PD5: MPN (none) -> CRCW0805100KFKEA
- R_LED1, R_LED2, R_LED3, R_LED4, R_LED5: MPN (none) -> CRCW08051K00FKEA
- R_SDP1, R_SDP2, R_SDP3, R_SDP4, R_SDP5: MPN (none) -> CRCW080510K0FKEA
- U_SD: MPN (none) -> TLV75533PDBVR
