File: hardware/pcb/interposer/interposer.kicad_pcb (KiCad board)
At the start: 2 copper layers, 67.1 x 46 mm, 35 parts, among them J1 POWER IN + / -, J2 40-pin stacking socket, J3 S+ / S- / VBUS / GND, J4 GND / PiTX / PiRX / MARK / Pi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, Q1 NMOS input, Q2 NMOS output, U1 LTC4367 protection switch, U2 UART power-off buffer

Commit message: still working on it
Parts:
- C1: footprint PicoPower:R_0805 -> PicoPower:C_0805_KEMET
- C2: value 100nF X7R 63V -> 100nF X7R 100V; footprint PicoPower:R_0805 -> PicoPower:C_0805_Murata
- C3, C4: footprint PicoPower:C_0805 -> PicoPower:C_0805_Murata
- R2, R3, R4: footprint PicoPower:R_0805 -> PicoPower:R_0805_TNPW
