File: hardware/pcb/interposer/interposer.kicad_pcb (KiCad board)
At the start: 2 copper layers, 67.1 x 46 mm, 35 parts, among them J1 POWER IN + / -, J2 40-pin stacking socket, J3 S+ / S- / VBUS / GND, J4 GND / PiTX / PiRX / MARK / Pi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, Q1 NMOS input, Q2 NMOS output, U1 LTC4367 protection switch, U2 UART power-off buffer

Commit message: Add the Phoenix fastening holes to the power header J1
Two 2.4 mm non-plated holes at board positions (3.82, 9.50) and (19.26, 9.50),
5.18 mm beyond the end pins and 2.5 mm from the pin row, per the Phoenix family
drawing, so the screwed plug's pull is carried by screws instead of the soldered
pins. The surrounding copper is ground only.

Two isolated ground stitching vias and one 0.2 mm ground track on B.Cu were
inside the hole clearance and are removed; native ERC, DRC and parity report 0
violations and 0 unconnected items, and nothing else changed (checked by
comparing tracks, vias and footprint positions). The correction lives in
footprint_corrections.phoenix_flange, shared with layout-interposer.py, and a
test checks the holes. The fastening screws are added to the BOM as a proposal,
the assembly steps and mechanical notes mention them, and the review files and
checklist are refreshed.

Co-Authored-By: Claude Sonnet 5.5 <noreply@anthropic.com>
Routing:
- net /GND: track 262.4 -> 248.1 mm, vias 99 -> 97
Changed lines of the file:
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@@
 			)
 		)
+		(pad "" np_thru_hole circle
+			(at -5.18 2.5 180)
+			(size 2.4 2.4)
+			(drill 2.4)
+			(layers "*.Cu" "*.Mask")
+		)
+		(pad "" np_thru_hole circle
+			(at 10.26 2.5 180)
+			(size 2.4 2.4)
+			(drill 2.4)
+			(layers "*.Cu" "*.Mask")
+		)
 		(pad "1" thru_hole roundrect
 			(at 0 0 180)
@@
 	)
 	(via
-		(at 3 11)
-		(size 0.6)
-		(drill 0.3)
-		(layers "F.Cu" "B.Cu")
-		(net 6)
-	)
-	(via
 		(at 19 7)
 		(size 0.6)
@@
 	)
 	(via
-		(at 19 11)
-		(size 0.6)
-		(drill 0.3)
-		(layers "F.Cu" "B.Cu")
-		(net 6)
-	)
-	(via
 		(at 7 7)
 		(size 0.6)
@@
 		(width 0.2)
 		(layer "B.Cu")
-		(net 6)
-	)
-	(segment
-		(start 28.3 9.7)
-		(end 14 9.7)
-		(width 0.2)
-		(layer "B.Cu")
