File: hardware/pcb/interposer/interposer.kicad_sch (KiCad schematic)
At the start: 34 parts, among them J1 POWER IN + / -, J2 40-pin stacking socket, J3 S+ / S- / VBUS / GND, J4 GND / PiTX / PiRX / MARK / Pi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, J5 Logical HAT side of J2, Q1 NMOS input, Q2 NMOS output, U1 LTC4367 protection switch, U2 UART power-off buffer

Commit message: still working on it
Parts:
- C1: footprint PicoPower:R_0805 -> PicoPower:C_0805_KEMET; MPN (none) -> C0805C123J5GACTU
- C2: value 100nF X7R 63V -> 100nF X7R 100V; footprint PicoPower:R_0805 -> PicoPower:C_0805_Murata; MPN (none) -> GRM21BR72A104JAC4L
- C3, C4: footprint PicoPower:C_0805 -> PicoPower:C_0805_Murata; MPN (none) -> GRM21BR71C104KA01L
- D1: MPN (none) -> APT2012LZGCK
- F1: MPN (none) -> 0031.8201
- J1: MPN (none) -> 1776508
- J2: MPN (none) -> SSQ-120-03-G-D
- J3: MPN (none) -> B4B-XH-A(LF)(SN)
- J4: MPN (none) -> B5B-XH-A(LF)(SN)
- Q1, Q2: MPN (none) -> BSC010N04LS6ATMA1
- R10, R11, R12, R13, R14, R15: MPN (none) -> CRCW0805100KFKEA
- R2: footprint PicoPower:R_0805 -> PicoPower:R_0805_TNPW; MPN (none) -> TNPW080510K0BEEA
- R3: footprint PicoPower:R_0805 -> PicoPower:R_0805_TNPW; MPN (none) -> TNPW08051K50BEEA
- R4: footprint PicoPower:R_0805 -> PicoPower:R_0805_TNPW; MPN (none) -> TNPW080595K3BEEA
- R5: MPN (none) -> CRCW0805510KFKEA
- R6, R7: MPN (none) -> CRCW080510R0FKEA
- R8: MPN (none) -> CRCW08055K10FKEA
- R9: MPN (none) -> CRCW08052K70FKEA
- RSH1: MPN (none) -> WSK25125L000DEA
- U1: MPN (none) -> LTC4367IMS8#PBF
- U2: MPN (none) -> SN74AXC4T245PWR
